File: PCB/Macropad.kicad_pcb (KiCad board)
At the start: 2 copper layers, 61.8 x 61.7 mm, 9 parts, among them SW1 SW_Push, SW2 SW_Push, SW3 SW_Push, SW4 SW_Push, SW5 SW_Push, SW6 SW_Push, U1 XAIO HERE

Commit message: OLED
Parts:
- added C1: 1 µF, Capacitor_SMD:C_0402_1005Metric, F.Cu at (143.6, 70.9)
- added DS1: OLED-128O064D, Display:OLED-128O064D, F.Cu at (138.6, 63.7)
- added R1: 910kΩ, Resistor_THT:R_Axial_DIN0204_L3.6mm_D1.6mm_P1.90mm_Vertical, F.Cu at (143.0, 66.8)
- U1: value XAIO HERE -> XIAO-RP2040-DIP
Connections:
- U1 pad 6: unconnected-(U1-GPIO7/SCL-Pad6) -> Net-(DS1-D1)
- U1 pad 7: unconnected-(U1-GPIO0/TX-Pad7) -> Net-(DS1-D0)
Routing:
- net Net-(DS1-D1): track 0.00 -> 195.7 mm, vias 0 -> 3
- net GND: track 182.4 -> 299.9 mm, vias 0 -> 1
- net Net-(DS1-D0): track 0.00 -> 61.1 mm, vias 0 -> 2
- net Net-(DS1-VCC): track 0.00 -> 9.22 mm
- net +3.3V: track 0.00 -> 7.19 mm
- net Net-(U1-GPIO27/ADC1/A1): track 71.9 -> 76.2 mm
- net Net-(D1-DIN): track 211.5 -> 207.8 mm
- net Net-(DS1-IREF): track 0.00 -> 3.53 mm
Other:
- board text added: "Xaio here"
